Commit message: new hand ball

File: humanoidverse/data/robots/h1/h1.urdf (robot description, URDF)
Before this commit: robot h1, 20 links, 19 joints
Links:
- added link left_hand_sphere; collision sphere radius=0.2; visual sphere radius=0.1
- added link right_hand_sphere; collision sphere radius=0.2; visual sphere radius=0.1
Joints:
- added joint left_hand_sphere_joint: type fixed, parent left_elbow_link, child left_hand_sphere, origin xyz=0 0 0 rpy=0 0 0
- added joint right_hand_sphere_joint: type fixed, parent right_elbow_link, child right_hand_sphere, origin xyz=0 0 0 rpy=0 0 0

Commit message: debug model

File: humanoidverse/data/robots/h1/h1.urdf (robot description, URDF)
Before this commit: robot h1, 22 links, 21 joints
Links:
- removed link left_hand_sphere
- removed link right_hand_sphere
Joints:
- removed joint left_hand_sphere_joint
- removed joint right_hand_sphere_joint
